File: LED-grid.kicad_sch (KiCad schematic)
At the start: 0 parts

Commit message: Finished schematic
Parts:
- added BT1: 6V, symbol Device:Battery
- added D1, D10, D100, D101, D102, D103, D104, D105, D106, D107, D108, D109, D11, D110, D111, D112, D113, D114, D115, D116, D117, D118, D119, D12, D120, D121, D122, D123, D124, D125, D126, D127, D128, D129, D13, D130, D131, D132, D133, D134, D135, D136, D137, D138, D139, D14, D140, D141, D142, D143, D144, D145, D146, D147, D148, D149, D15, D150, D151, D152, D153, D154, D155, D156, D157, D158, D159, D16, D160, D161, D162, D163, D164, D165, D166, D167, D168, D169, D17, D170, D171, D172, D173, D174, D175, D176, D177, D178, D179, D18, D180, D181, D182, D183, D184, D185, D186, D187, D188, D189, D19, D190, D191, D192, D193, D194, D195, D196, D197, D198, D199, D2, D20, D200, D201, D202, D203, D204, D205, D206, D207, D208, D209, D21, D210, D211, D212, D213, D214, D215, D216, D217, D218, D219, D22, D220, D221, D222, D223, D224, D225, D23, D24, D25, D26, D27, D28, D29, D3, D30, D31, D32, D33, D34, D35, D36, D37, D38, D39, D4, D40, D41, D42, D43, D44, D45, D46, D47, D48, D49, D5, D50, D51, D52, D53, D54, D55, D56, D57, D58, D59, D6, D60, D61, D62, D63, D64, D65, D66, D67, D68, D69, D7, D70, D71, D72, D73, D74, D75, D76, D77, D78, D79, D8, D80, D81, D82, D83, D84, D85, D86, D87, D88, D89, D9, D90, D91, D92, D93, D94, D95, D96, D97, D98, D99: LED, LED_SMD:LED_0603_1608Metric, symbol Device:LED
- added R1, R10, R11, R12, R13, R14, R15, R16, R17, R18, R19, R2, R20, R21, R22, R23, R24, R25, R26, R27, R28, R29, R3, R30, R31, R32, R33, R34, R35, R36, R37, R38, R39, R4, R40, R41, R42, R43, R44, R45, R46, R47, R48, R49, R5, R50, R51, R52, R53, R54, R55, R56, R57, R58, R59, R6, R60, R61, R62, R63, R64, R65, R66, R67, R68, R69, R7, R70, R71, R72, R73, R74, R75, R8, R9: 120, Resistor_SMD:R_0805_2012Metric, symbol Device:R
Connections:
- new net: D111.1 (K), D126.2 (A)
- new net: D111.2 (A), D96.1 (K)
- new net: D220.1 (K), R70.1
- new net: D41.1 (K), R11.1
- new net: D193.1 (K), D208.2 (A)
- new net: D201.1 (K), D216.2 (A)
- new net: D186.1 (K), D201.2 (A)
- new net: D172.1 (K), R52.1
- new net: D157.1 (K), D172.2 (A)
- new net: D55.1 (K), D70.2 (A)
- new net: D113.2 (A), D98.1 (K)
- new net: D27.1 (K), R7.1
- new net: D22.1 (K), D27.2 (A)
- new net: D151.1 (K), D166.2 (A)
- new net: D136.1 (K), D151.2 (A)
- new net: D54.1 (K), D69.2 (A)
- new net: D150.1 (K), D165.2 (A)
- new net: D7.1 (K), D8.2 (A)
- new net: D128.1 (K), R38.1
- new net: D113.1 (K), D128.2 (A)
- new net: D135.1 (K), R45.1
- new net: D120.1 (K), D135.2 (A)
- new net: D188.1 (K), D203.2 (A)
- new net: D102.1 (K), D117.2 (A)
- new net: D45.1 (K), R15.1
- new net: D17.1 (K), D22.2 (A)
- new net: D83.1 (K), R23.1
- new net: D68.1 (K), D83.2 (A)
- new net: D184.1 (K), D199.2 (A)
- new net: D212.1 (K), R62.1
- new net: D105.1 (K), D120.2 (A)
- new net: D210.1 (K), D225.2 (A)
- new net: D195.1 (K), D210.2 (A)
- new net: D204.1 (K), D219.2 (A)
- new net: D189.1 (K), D204.2 (A)
- new net: D121.1 (K), R31.1
- new net: D106.1 (K), D121.2 (A)
- new net: D131.1 (K), R41.1
- new net: D116.1 (K), D131.2 (A)
- new net: D67.1 (K), D82.2 (A)
- new net: D52.1 (K), D67.2 (A)
- new net: D51.1 (K), D66.2 (A)
- new net: D46.1 (K), D61.2 (A)
- new net: D217.1 (K), R67.1
- new net: D202.1 (K), D217.2 (A)
- new net: D85.1 (K), R25.1
- new net: D70.1 (K), D85.2 (A)
- new net: D224.1 (K), R74.1
- new net: D118.1 (K), D133.2 (A)
- new net: D103.1 (K), D118.2 (A)
- new net: D49.1 (K), D64.2 (A)
- new net: D124.1 (K), R34.1
- new net: D36.1 (K), D41.2 (A)
- new net: D31.1 (K), D36.2 (A)
- new net: D84.1 (K), R24.1
- new net: D69.1 (K), D84.2 (A)
- new net: D209.1 (K), D224.2 (A)
- new net: D194.1 (K), D209.2 (A)
- new net: D71.1 (K), D86.2 (A)
- new net: D56.1 (K), D71.2 (A)
- new net: D86.1 (K), R26.1
- new net: D23.1 (K), D28.2 (A)
- new net: D18.1 (K), D23.2 (A)
- new net: D80.1 (K), R20.1
- new net: D65.1 (K), D80.2 (A)
- new net: D175.1 (K), R55.1
- new net: D191.1 (K), D206.2 (A)
- new net: D176.1 (K), R56.1
- new net: D161.1 (K), D176.2 (A)
- new net: D30.1 (K), R10.1
- new net: D25.1 (K), D30.2 (A)
- new net: D213.1 (K), R63.1
- new net: D34.1 (K), D39.2 (A)
- new net: D15.1 (K), R5.1
- new net: D168.1 (K), R48.1
- new net: D155.1 (K), D170.2 (A)
- new net: D140.1 (K), D155.2 (A)
- new net: D3.1 (K), R1.1
- new net: D2.1 (K), D3.2 (A)
- new net: D44.1 (K), R14.1
- new net: D39.1 (K), D44.2 (A)
- new net: D100.1 (K), D115.2 (A)
- new net: D48.1 (K), D63.2 (A)
- new net: D173.1 (K), R53.1
- new net: D219.1 (K), R69.1
- new net: D123.1 (K), R33.1
- new net: D108.1 (K), D123.2 (A)
- new net: D81.1 (K), R21.1
- new net: D137.1 (K), D152.2 (A)
- new net: D205.1 (K), D220.2 (A)
- new net: D177.1 (K), R57.1
- new net: D162.1 (K), D177.2 (A)
- new net: D82.1 (K), R22.1
- new net: D42.1 (K), R12.1
- new net: D223.1 (K), R73.1
- new net: D216.1 (K), R66.1
- new net: D134.1 (K), R44.1
- new net: D119.1 (K), D134.2 (A)
- new net: D211.1 (K), R61.1
- new net: D196.1 (K), D211.2 (A)
- new net: D197.1 (K), D212.2 (A)
- new net: D166.1 (K), R46.1
- new net: D179.1 (K), R59.1
- new net: D74.1 (K), D89.2 (A)
- new net: D59.1 (K), D74.2 (A)
- new net: D144.1 (K), D159.2 (A)
- new net: D4.1 (K), D5.2 (A)
- new net: D66.1 (K), D81.2 (A)
- new net: D10.1 (K), D11.2 (A)
- new net: D203.1 (K), D218.2 (A)
- new net: D110.1 (K), D125.2 (A)
- new net: D110.2 (A), D95.1 (K)
- new net: D156.1 (K), D171.2 (A)
- new net: D141.1 (K), D156.2 (A)
- new net: D214.1 (K), R64.1
- new net: D199.1 (K), D214.2 (A)
- new net: D107.1 (K), D122.2 (A)
- new net: D107.2 (A), D92.1 (K)
- new net: D180.1 (K), R60.1
- new net: D165.1 (K), D180.2 (A)
- new net: D122.1 (K), R32.1
- new net: D33.1 (K), D38.2 (A)
- new net: D153.1 (K), D168.2 (A)
- new net: D138.1 (K), D153.2 (A)
- new net: D147.1 (K), D162.2 (A)
- new net: D117.1 (K), D132.2 (A)
- new net: D142.1 (K), D157.2 (A)
- new net: D125.1 (K), R35.1
- new net: D178.1 (K), R58.1
- new net: D163.1 (K), D178.2 (A)
- new net: D50.1 (K), D65.2 (A)
- new net: D215.1 (K), R65.1
- new net: D106.2 (A), D91.1 (K)
- new net: D182.1 (K), D197.2 (A)
- new net: D160.1 (K), D175.2 (A)
- new net: D190.1 (K), D205.2 (A)
- new net: D183.1 (K), D198.2 (A)
- new net: D38.1 (K), D43.2 (A)
- new net: D1.1 (K), D2.2 (A)
- new net: D133.1 (K), R43.1
- new net: D90.1 (K), R30.1
- new net: D200.1 (K), D215.2 (A)
- new net: D57.1 (K), D72.2 (A)
- new net: D112.1 (K), D127.2 (A)
- new net: D112.2 (A), D97.1 (K)
- new net: D146.1 (K), D161.2 (A)
- new net: D174.1 (K), R54.1
- new net: D9.1 (K), R3.1
- new net: D16.1 (K), D21.2 (A)
- new net: D192.1 (K), D207.2 (A)
- new net: D198.1 (K), D213.2 (A)
- new net: D13.1 (K), D14.2 (A)
- new net: D37.1 (K), D42.2 (A)
- new net: D32.1 (K), D37.2 (A)
- new net: D158.1 (K), D173.2 (A)
- new net: D143.1 (K), D158.2 (A)
- new net: D132.1 (K), R42.1
- new net: D225.1 (K), R75.1
- new net: D108.2 (A), D93.1 (K)
- new net: D152.1 (K), D167.2 (A)
- new net: D170.1 (K), R50.1
- new net: D167.1 (K), R47.1
- new net: D75.1 (K), D90.2 (A)
- new net: D60.1 (K), D75.2 (A)
- new net: D101.1 (K), D116.2 (A)
- new net: D26.1 (K), R6.1
- new net: D21.1 (K), D26.2 (A)
- new net: D72.1 (K), D87.2 (A)
- new net: D14.1 (K), D15.2 (A)
- new net: D185.1 (K), D200.2 (A)
- new net: D127.1 (K), R37.1
- new net: D159.1 (K), D174.2 (A)
- new net: D221.1 (K), R71.1
- new net: D206.1 (K), D221.2 (A)
- new net: D6.1 (K), R2.1
- new net: D5.1 (K), D6.2 (A)
- new net: D89.1 (K), R29.1
- new net: D12.1 (K), R4.1
- new net: D88.1 (K), R28.1
- new net: D73.1 (K), D88.2 (A)
- new net: D148.1 (K), D163.2 (A)
- new net: D87.1 (K), R27.1
- new net: D139.1 (K), D154.2 (A)
- new net: D109.2 (A), D94.1 (K)
- new net: D62.1 (K), D77.2 (A)
- new net: D47.1 (K), D62.2 (A)
- new net: D187.1 (K), D202.2 (A)
- new net: D130.1 (K), R40.1
- new net: D115.1 (K), D130.2 (A)
- new net: D20.1 (K), D25.2 (A)
- new net: D58.1 (K), D73.2 (A)
- new net: D169.1 (K), R49.1
- new net: D154.1 (K), D169.2 (A)
- new net: D78.1 (K), R18.1
- new net: D164.1 (K), D179.2 (A)
- new net: D24.1 (K), D29.2 (A)
- new net: D19.1 (K), D24.2 (A)
- new net: D218.1 (K), R68.1
- new net: D53.1 (K), D68.2 (A)
- new net: D171.1 (K), R51.1
- new net: D63.1 (K), D78.2 (A)
- new net: D11.1 (K), D12.2 (A)
- new net: D77.1 (K), R17.1
- new net: D61.1 (K), D76.2 (A)
- new net: D126.1 (K), R36.1
- new net: D40.1 (K), D45.2 (A)
- new net: D35.1 (K), D40.2 (A)
- new net: D222.1 (K), R72.1
- new net: D207.1 (K), D222.2 (A)
- new net: D104.1 (K), D119.2 (A)
- new net: D208.1 (K), D223.2 (A)
- new net: D109.1 (K), D124.2 (A)
- new net: D43.1 (K), R13.1
- new net: D145.1 (K), D160.2 (A)
- new net: D149.1 (K), D164.2 (A)
- new net: D29.1 (K), R9.1
- new net: D114.1 (K), D129.2 (A)
- new net: D114.2 (A), D99.1 (K)
- new net: D181.1 (K), D196.2 (A)
- new net: D64.1 (K), D79.2 (A)
- new net: D76.1 (K), R16.1
- new net: D79.1 (K), R19.1
- new net: D28.1 (K), R8.1
- new net: D129.1 (K), R39.1
- new net: D8.1 (K), D9.2 (A)
- new net GND: BT1.2 (-), R1.2, R10.2, R11.2, R12.2, R13.2, R14.2, R15.2, R16.2, R17.2, R18.2, R19.2, R2.2, R20.2, R21.2, R22.2, R23.2, R24.2, R25.2, R26.2, R27.2, R28.2, R29.2, R3.2, R30.2, R31.2, R32.2, R33.2, R34.2, R35.2, R36.2, R37.2, R38.2, R39.2, R4.2, R40.2, R41.2, R42.2, R43.2, R44.2, R45.2, R46.2, R47.2, R48.2, R49.2, R5.2, R50.2, R51.2, R52.2, R53.2, R54.2, R55.2, R56.2, R57.2, R58.2, R59.2, R6.2, R60.2, R61.2, R62.2, R63.2, R64.2, R65.2, R66.2, R67.2, R68.2, R69.2, R7.2, R70.2, R71.2, R72.2, R73.2, R74.2, R75.2, R8.2, R9.2
- new net VCC: BT1.1 (+), D1.2 (A), D10.2 (A), D100.2 (A), D101.2 (A), D102.2 (A), D103.2 (A), D104.2 (A), D105.2 (A), D13.2 (A), D136.2 (A), D137.2 (A), D138.2 (A), D139.2 (A), D140.2 (A), D141.2 (A), D142.2 (A), D143.2 (A), D144.2 (A), D145.2 (A), D146.2 (A), D147.2 (A), D148.2 (A), D149.2 (A), D150.2 (A), D16.2 (A), D17.2 (A), D18.2 (A), D181.2 (A), D182.2 (A), D183.2 (A), D184.2 (A), D185.2 (A), D186.2 (A), D187.2 (A), D188.2 (A), D189.2 (A), D19.2 (A), D190.2 (A), D191.2 (A), D192.2 (A), D193.2 (A), D194.2 (A), D195.2 (A), D20.2 (A), D31.2 (A), D32.2 (A), D33.2 (A), D34.2 (A), D35.2 (A), D4.2 (A), D46.2 (A), D47.2 (A), D48.2 (A), D49.2 (A), D50.2 (A), D51.2 (A), D52.2 (A), D53.2 (A), D54.2 (A), D55.2 (A), D56.2 (A), D57.2 (A), D58.2 (A), D59.2 (A), D60.2 (A), D7.2 (A), D91.2 (A), D92.2 (A), D93.2 (A), D94.2 (A), D95.2 (A), D96.2 (A), D97.2 (A), D98.2 (A), D99.2 (A)
Other:
- title: (none) -> LED Panel

Commit message: Updated battery footprint
Parts:
- BT1: footprint (none) -> Connector_PinHeader_1.00mm:PinHeader_1x02_P1.00mm_Vertical
Changed lines of the file:
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@@
 			)
 		)
-		(property "Footprint" ""
+		(property "Footprint" "Connector_PinHeader_1.00mm:PinHeader_1x02_P1.00mm_Vertical"
 			(at 16.51 22.606 90)
 			(effects

Commit message: Finished laying out PCB
Parts:
- renumbered D94 to D100, D109 to D101, D124 to D102, D95 to D103, D110 to D104, D125 to D105, D96 to D106, D111 to D107, D126 to D108, D97 to D109, D112 to D110, D127 to D111, D98 to D112, D128 to D114, D99 to D115, D114 to D116, D129 to D117, D100 to D118, D115 to D119, D130 to D120, D101 to D121, D116 to D122, D131 to D123, D102 to D124, D117 to D125, D132 to D126, D103 to D127, D118 to D128, D133 to D129, D104 to D130, D119 to D131, D134 to D132, D105 to D133, D120 to D134, D151 to D137, D166 to D138, D137 to D139, D152 to D140, D167 to D141, D138 to D142, D153 to D143, D168 to D144, D139 to D145, D154 to D146, D169 to D147, D140 to D148, D155 to D149, D170 to D150, D141 to D151, D156 to D152, D171 to D153, D142 to D154, D157 to D155, D172 to D156, D143 to D157, D173 to D159, D144 to D160, D159 to D161, D174 to D162, D145 to D163, D160 to D164, D175 to D165, D146 to D166, D161 to D167, D176 to D168, D147 to D169, D21 to D17, D162 to D170, D177 to D171, D148 to D172, D163 to D173, D178 to D174, D149 to D175, D164 to D176, D179 to D177, D150 to D178, D165 to D179, D26 to D18, D196 to D182, D211 to D183, D182 to D184, D197 to D185, D212 to D186, D183 to D187, D198 to D188, D213 to D189, D17 to D19, D184 to D190, D199 to D191, D214 to D192, D185 to D193, D200 to D194, D215 to D195, D186 to D196, D201 to D197, D216 to D198, D187 to D199, D22 to D20, D202 to D200, D217 to D201, D188 to D202, D218 to D204, D189 to D205, D204 to D206, D219 to D207, D190 to D208, D205 to D209, D27 to D21, D220 to D210, D191 to D211, D206 to D212, D221 to D213, D192 to D214, D207 to D215, D222 to D216, D193 to D217, D208 to D218, D223 to D219, D18 to D22, D194 to D220, D209 to D221, D224 to D222, D195 to D223, D210 to D224, D28 to D24, D19 to D25, D24 to D26, D29 to D27, D20 to D28, D25 to D29, D36 to D32, D41 to D33, D32 to D34, D37 to D35, D42 to D36, D33 to D37, D43 to D39, D34 to D40, D39 to D41, D44 to D42, D35 to D43, D40 to D44, D61 to D47, D76 to D48, D47 to D49, D62 to D50, D77 to D51, D48 to D52, D63 to D53, D78 to D54, D49 to D55, D64 to D56, D79 to D57, D50 to D58, D65 to D59, D80 to D60, D51 to D61, D66 to D62, D81 to D63, D52 to D64, D67 to D65, D82 to D66, D53 to D67, D83 to D69, D54 to D70, D69 to D71, D84 to D72, D55 to D73, D70 to D74, D85 to D75, D56 to D76, D71 to D77, D86 to D78, D57 to D79, D72 to D80, D87 to D81, D58 to D82, D73 to D83, D88 to D84, D59 to D85, D74 to D86, D89 to D87, D60 to D88, D75 to D89, D106 to D92, D121 to D93, D92 to D94, D107 to D95, D122 to D96, D93 to D97, D108 to D98, D123 to D99

Commit message: Version 1.0.1 We can now actually control the brightness using a potentiometer
Parts:
- added C1: 10n, Capacitor_SMD:C_0603_1608Metric, symbol Device:C
- added C2: 100n, Capacitor_SMD:C_0402_1005Metric, symbol Device:C
- added Q1: NMOS, Package_TO_SOT_THT:TO-220-3_Horizontal_TabUp, symbol Simulation_SPICE:NMOS
- added R76, R77, R78, R79: 1k, Resistor_SMD:R_0805_2012Metric, symbol Device:R
- added RV1: 3296X-1-102LF, Potentiometer_THT:Potentiometer_Bourns_3296X_Horizontal, symbol Device:R_Potentiometer
- added SW1: SW_Wuerth_450301014042, Button_Switch_THT:SW_Slide_SPDT_Angled_CK_OS102011MA1Q, symbol Switch:SW_Wuerth_450301014042
- added U1: NE555D, Package_SO:SOIC-8_3.9x4.9mm_P1.27mm, symbol Timer:NE555D
- added U2: LM741, Package_SO:SOIC-8_3.9x4.9mm_P1.27mm, symbol Amplifier_Operational:LM741
- BT1: footprint Connector_PinHeader_1.00mm:PinHeader_1x02_P1.00mm_Vertical -> Connector_JST:JST_EH_B2B-EH-A_1x02_P2.50mm_Vertical
Connections:
- net GND: now also C1.2, C2.2, R78.1, SW1.3 (A), U1.1 (GND), U1.7 (DIS), U2.4 (V-)
- net VCC: now also Q1.1 (D), R77.2, SW1.1 (B), U1.4 (R), U1.8 (VCC), U2.7 (V+); no longer BT1.1 (+), D1.2 (A), D10.2 (A), D100.2 (A), D103.2 (A), D106.2 (A), D109.2 (A), D112.2 (A), D115.2 (A), D118.2 (A), D121.2 (A), D124.2 (A), D127.2 (A), D13.2 (A), D130.2 (A), D133.2 (A), D136.2 (A), D139.2 (A), D142.2 (A), D145.2 (A), D148.2 (A), D151.2 (A), D154.2 (A), D157.2 (A), D16.2 (A), D160.2 (A), D163.2 (A), D166.2 (A), D169.2 (A), D172.2 (A), D175.2 (A), D178.2 (A), D181.2 (A), D184.2 (A), D187.2 (A), D19.2 (A), D190.2 (A), D193.2 (A), D196.2 (A), D199.2 (A), D202.2 (A), D205.2 (A), D208.2 (A), D211.2 (A), D214.2 (A), D217.2 (A), D22.2 (A), D220.2 (A), D223.2 (A), D25.2 (A), D28.2 (A), D31.2 (A), D34.2 (A), D37.2 (A), D4.2 (A), D40.2 (A), D43.2 (A), D46.2 (A), D49.2 (A), D52.2 (A), D55.2 (A), D58.2 (A), D61.2 (A), D64.2 (A), D67.2 (A), D7.2 (A), D70.2 (A), D73.2 (A), D76.2 (A), D79.2 (A), D82.2 (A), D85.2 (A), D88.2 (A), D91.2 (A), D94.2 (A), D97.2 (A)
- new net: R77.1, RV1.1
- new net: RV1.2, U2.3 (+)
- new net: R78.2, RV1.3
- new net: Q1.2 (G), R79.2
- new net: R76.1, U1.3 (Q)
- new net: C2.1, R76.2, U1.2 (TR), U1.6 (THR), U2.2 (-)
- new net: R79.1, U2.6
- new net: C1.1, U1.5 (CV)
- new net: BT1.1 (+), SW1.2 (C)
- new net LED_PWR: D1.2 (A), D10.2 (A), D100.2 (A), D103.2 (A), D106.2 (A), D109.2 (A), D112.2 (A), D115.2 (A), D118.2 (A), D121.2 (A), D124.2 (A), D127.2 (A), D13.2 (A), D130.2 (A), D133.2 (A), D136.2 (A), D139.2 (A), D142.2 (A), D145.2 (A), D148.2 (A), D151.2 (A), D154.2 (A), D157.2 (A), D16.2 (A), D160.2 (A), D163.2 (A), D166.2 (A), D169.2 (A), D172.2 (A), D175.2 (A), D178.2 (A), D181.2 (A), D184.2 (A), D187.2 (A), D19.2 (A), D190.2 (A), D193.2 (A), D196.2 (A), D199.2 (A), D202.2 (A), D205.2 (A), D208.2 (A), D211.2 (A), D214.2 (A), D217.2 (A), D22.2 (A), D220.2 (A), D223.2 (A), D25.2 (A), D28.2 (A), D31.2 (A), D34.2 (A), D37.2 (A), D4.2 (A), D40.2 (A), D43.2 (A), D46.2 (A), D49.2 (A), D52.2 (A), D55.2 (A), D58.2 (A), D61.2 (A), D64.2 (A), D67.2 (A), D7.2 (A), D70.2 (A), D73.2 (A), D76.2 (A), D79.2 (A), D82.2 (A), D85.2 (A), D88.2 (A), D91.2 (A), D94.2 (A), D97.2 (A), Q1.3 (S)
Other:
- note added: "Brightness Regulation"
- note added: "LED Panel"
- note added: "ON/OFF Switch"
- moved on the sheet: BT1, D1, D10, D100, D101, D102, D103, D104, D105, D106, D107, D108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

Commit message: Updated schematic
Parts:
- removed BT1: 6V, Connector_JST:JST_EH_B2B-EH-A_1x02_P2.50mm_Vertical, symbol Device:Battery
- removed D2: LED, LED_SMD:LED_0603_1608Metric, symbol Device:LED
- removed Q1: NMOS, Package_TO_SOT_THT:TO-220-3_Horizontal_TabUp, symbol Simulation_SPICE:NMOS
- removed R35, R36, R37, R38, R39, R40, R41, R42, R43, R44, R45, R46, R47, R48, R49, R50, R51, R52, R53, R54, R55, R56, R57, R58, R59, R60, R61, R62, R63, R64, R65, R66, R67, R68, R69, R70, R71, R72, R73, R74, R75: 120, Resistor_SMD:R_0805_2012Metric, symbol Device:R
- removed R76, R77, R78, R79: 1k, Resistor_SMD:R_0805_2012Metric, symbol Device:R
- removed U1: NE555D, Package_SO:SOIC-8_3.9x4.9mm_P1.27mm, symbol Timer:NE555D
- removed U2: LM741, Package_SO:SOIC-8_3.9x4.9mm_P1.27mm, symbol Amplifier_Operational:LM741
- added C3, C4, C5: 1u, Capacitor_SMD:C_0603_1608Metric, symbol Device:C
- added C6: 10n, Capacitor_SMD:C_0603_1608Metric, symbol Device:C
- added C7: 1n, Capacitor_SMD:C_0201_0603Metric, symbol Device:C
- added C8: 2u, Capacitor_SMD:C_0603_1608Metric, symbol Device:C
- added C9: 47n, Capacitor_SMD:C_0201_0603Metric, symbol Device:C
- added D2: D, Diode_SMD:D_0603_1608Metric, symbol Device:D
- added D226, D227: LED, LED_SMD:LED_0603_1608Metric, symbol Device:LED
- added J1: Conn_01x03_Pin, Connector_JST:JST_ZH_B3B-ZR_1x03_P1.50mm_Vertical, symbol Connector:Conn_01x03_Pin
- added J2: USB_C_Receptacle, Connector_USB:USB_C_Receptacle_Amphenol_12401610E4-2A, symbol Connector:USB_C_Receptacle
- added L1: 30u, symbol Device:L
- added U1: TPS923650D2DRLR, symbol custom:TPS923650D2DRLR
- added U3: BQ24052, symbol custom:BQ24052
- C1: value 10n -> 1u
- C2: value 100n -> 1u; footprint Capacitor_SMD:C_0402_1005Metric -> Capacitor_SMD:C_0603_1608Metric
- R1, R2: value 120 -> 5.1k; footprint Resistor_SMD:R_0805_2012Metric -> (none)
- R10, R11, R12, R13, R14, R15, R16, R17, R18, R19, R20, R21, R22, R23, R24, R25, R26, R27, R28, R29, R30, R31, R32, R33, R34: value 120 -> 20; footprint Resistor_SMD:R_0805_2012Metric -> Resistor_SMD:R_0201_0603Metric
- R3, R4, R6: value 120 -> 1k; footprint Resistor_SMD:R_0805_2012Metric -> (none)
- R5: value 120 -> 2k; footprint Resistor_SMD:R_0805_2012Metric -> (none)
- R7, R8: value 120 -> 100; footprint Resistor_SMD:R_0805_2012Metric -> Resistor_SMD:R_0201_0603Metric
- R9: value 120 -> 1.6; footprint Resistor_SMD:R_0805_2012Metric -> Resistor_SMD:R_0201_0603Metric
- RV1: value 3296X-1-102LF -> 1k
- SW1: footprint Button_Switch_THT:SW_Slide_SPDT_Angled_CK_OS102011MA1Q -> Button_Switch_THT:SW_NKK_G1xJP
Connections:
- net GND: now also R4.1, R5.1, RV1.3, SW1.2 (C), C3.1, C4.2, C5.2, C6.2, C9.2, J1.3 (Pin_3), J2.A1 (GND), J2.A12 (GND), J2.B1 (GND), J2.B12 (GND), U1.1 (GND), U1.9 (TP), U3.11 (TP), U3.3 (VSS), U3.7 (ISET2); no longer R3.2, R4.2, R5.2, R6.2, R7.2, R8.2, R9.2, SW1.3 (A)
- net LED_PWR: now also D102.2 (A), D111.2 (A), D12.2 (A), D120.2 (A), D129.2 (A), D138.2 (A), D147.2 (A), D156.2 (A), D165.2 (A), D174.2 (A), D183.2 (A), D192.2 (A), D201.2 (A), D21.2 (A), D210.2 (A), D219.2 (A), D3.2 (A), D30.2 (A), D39.2 (A), D48.2 (A), D57.2 (A), D66.2 (A), D75.2 (A), D84.2 (A), D93.2 (A), R8.2, R9.2, C8.2, C9.1; no longer D1.2 (A), D10.2 (A), D100.2 (A), D103.2 (A), D106.2 (A), D109.2 (A), D112.2 (A), D115.2 (A), D118.2 (A), D121.2 (A), D124.2 (A), D127.2 (A), D13.2 (A), D130.2 (A), D133.2 (A), D136.2 (A), D139.2 (A), D142.2 (A), D145.2 (A), D148.2 (A), D151.2 (A), D154.2 (A), D157.2 (A), D16.2 (A), D160.2 (A), D163.2 (A), D166.2 (A), D169.2 (A), D172.2 (A), D175.2 (A), D178.2 (A), D181.2 (A), D184.2 (A), D187.2 (A), D19.2 (A), D190.2 (A), D193.2 (A), D196.2 (A), D199.2 (A), D202.2 (A), D205.2 (A), D208.2 (A), D211.2 (A), D214.2 (A), D217.2 (A), D22.2 (A), D220.2 (A), D223.2 (A), D25.2 (A), D28.2 (A), D31.2 (A), D34.2 (A), D37.2 (A), D4.2 (A), D40.2 (A), D43.2 (A), D46.2 (A), D49.2 (A), D52.2 (A), D55.2 (A), D58.2 (A), D61.2 (A), D64.2 (A), D67.2 (A), D7.2 (A), D70.2 (A), D73.2 (A), D76.2 (A), D79.2 (A), D82.2 (A), D85.2 (A), D88.2 (A), D91.2 (A), D94.2 (A), D97.2 (A)
- net VCC: now also RV1.1, C4.1, L1.1, U1.2 (VIN)
- net at D210.1 (K): now also D211.2 (A)
- net at D33.1 (K): now also D34.2 (A); no longer R11.1
- net at D156.1 (K): now also D157.2 (A)
- net at D155.1 (K): now also R26.1; no longer D156.2 (A)
- net at D21.1 (K): now also D22.2 (A); no longer R7.1
- net at D20.1 (K): now also R11.1; no longer D21.2 (A)
- net at D137.1 (K): now also R24.1; no longer D138.2 (A)
- net at D114.1 (K): now also D115.2 (A)
- net at D135.1 (K): now also D136.2 (A)
- net at R15.1: now also D56.1 (K); no longer D45.1 (K)
- net at D69.1 (K): now also D70.2 (A); no longer R23.1
- net at D186.1 (K): now also D187.2 (A)
- net at D93.1 (K): now also D94.2 (A); no longer R31.1
- net at D92.1 (K): now also R19.1; no longer D93.2 (A)
- net at D123.1 (K): now also D124.2 (A)
- net at RV1.2: now also U1.3 (DIM)
- net at D65.1 (K): now also R16.1; no longer D66.2 (A)
- net at D201.1 (K): now also D202.2 (A)
- net at D200.1 (K): now also R31.1; no longer D201.2 (A)
- net at D75.1 (K): now also D76.2 (A); no longer R25.1
- net at D74.1 (K): now also R17.1; no longer D75.2 (A)
- net at D222.1 (K): now also D223.2 (A)
- net at D128.1 (K): now also R23.1; no longer D129.2 (A)
- net at D102.1 (K): now also D103.2 (A); no longer R34.1
- net at D72.1 (K): now also D73.2 (A); no longer R24.1
- net at D78.1 (K): now also D79.2 (A); no longer R26.1
- net at R20.1: now also D101.1 (K); no longer D60.1 (K)
- net at D165.1 (K): now also D166.2 (A)
- net at D168.1 (K): now also D169.2 (A)
- net at D30.1 (K): now also D31.2 (A); no longer R10.1
- net at D29.1 (K): now also R12.1; no longer D30.2 (A)
- net at D189.1 (K): now also D190.2 (A)
- net at D15.1 (K): now also D16.2 (A); no longer R5.1
- net at D144.1 (K): now also D145.2 (A)
- net at R1.1: now also J2.A5 (CC1); no longer D3.1 (K)
- net at R14.1: now also D47.1 (K); no longer D42.1 (K)
- net at D159.1 (K): now also D160.2 (A)
- net at D207.1 (K): now also D208.2 (A)
- net at R33.1: now also D218.1 (K); no longer D99.1 (K)
- net at D63.1 (K): now also D64.2 (A); no longer R21.1
- net at D209.1 (K): now also R32.1; no longer D210.2 (A)
- net at D171.1 (K): now also D172.2 (A)
- net at R22.1: now also D119.1 (K); no longer D66.1 (K)
- net at D36.1 (K): now also D37.2 (A); no longer R12.1
- net at D219.1 (K): now also D220.2 (A)
- net at D198.1 (K): now also D199.2 (A)
- net at D132.1 (K): now also D133.2 (A)
- net at D183.1 (K): now also D184.2 (A)
- net at D182.1 (K): now also R29.1; no longer D183.2 (A)
- net at D138.1 (K): now also D139.2 (A)
- net at D177.1 (K): now also D178.2 (A)
- net VBUS: now reaches C2.1
- net VBUS: now also J2.A4 (VBUS), J2.A9 (VBUS), J2.B4 (VBUS), J2.B9 (VBUS), U3.1 (IN)
- net at D192.1 (K): now also D193.2 (A)
- net at D191.1 (K): now also R30.1; no longer D192.2 (A)
- net at D180.1 (K): now also D181.2 (A)
- net at D96.1 (K): now also D97.2 (A); no longer R32.1
- net at D105.1 (K): now also D106.2 (A)
- net at D174.1 (K): now also D175.2 (A)
- net at D173.1 (K): now also R28.1; no longer D174.2 (A)
- net at D195.1 (K): now also D196.2 (A)
- net at D164.1 (K): now also R27.1; no longer D165.2 (A)
- net at D38.1 (K): now also R13.1; no longer D39.2 (A)
- net at D1.1 (K): now also U3.8 (CHG)
- net at D129.1 (K): now also D130.2 (A)
- net at D90.1 (K): now also D91.2 (A); no longer R30.1
- net at D110.1 (K): now also R21.1; no longer D111.2 (A)
- net at D162.1 (K): now also D163.2 (A)
- net at R3.1: now also J2.S1 (SHIELD); no longer D9.1 (K)
- net at D126.1 (K): now also D127.2 (A)
- net at D225.1 (K): now also D226.2 (A)
- net at D150.1 (K): now also D151.2 (A)
- net at D141.1 (K): now also D142.2 (A)
- net at D18.1 (K): now also D19.2 (A); no longer R6.1
- net at D111.1 (K): now also D112.2 (A)
- net at D213.1 (K): now also D214.2 (A)
- net at R2.1: now also J2.B5 (CC2); no longer D6.1 (K)
- net at D87.1 (K): now also D88.2 (A); no longer R29.1
- net at D12.1 (K): now also D13.2 (A); no longer R4.1
- net at D84.1 (K): now also D85.2 (A); no longer R28.1
- net at D83.1 (K): now also R18.1; no longer D84.2 (A)
- net at D81.1 (K): now also D82.2 (A); no longer R27.1
- net at D120.1 (K): now also D121.2 (A)
- net at D147.1 (K): now also D148.2 (A)
- net at D146.1 (K): now also R25.1; no longer D147.2 (A)
- net at D54.1 (K): now also D55.2 (A); no longer R18.1
- net at D204.1 (K): now also D205.2 (A)
- net at D153.1 (K): now also D154.2 (A)
- net at D11.1 (K): now also R10.1; no longer D12.2 (A)
- net at D51.1 (K): now also D52.2 (A); no longer R17.1
- net at D108.1 (K): now also D109.2 (A)
- net at D216.1 (K): now also D217.2 (A)
- net at D39.1 (K): now also D40.2 (A); no longer R13.1
- net at C1.1: now also R3.2
- net at D27.1 (K): now also D28.2 (A); no longer R9.1
- net at D48.1 (K): now also D49.2 (A); no longer R16.1
- net at D57.1 (K): now also D58.2 (A); no longer R19.1
- net at R8.1: now also C7.2, U1.6 (CSN); no longer D24.1 (K)
- net at D117.1 (K): now also D118.2 (A)
- new net: D3.1 (K), D4.2 (A)
- new net: D45.1 (K), D46.2 (A)
- new net: C6.1, R7.2
- new net: C7.1, C8.1, D2.1 (K), R9.1, U1.7 (CSP)
- new net: D2.2 (A), L1.2, U1.8 (SW)
- new net: D24.1 (K), D25.2 (A)
- new net: D60.1 (K), D61.2 (A)
- new net: D42.1 (K), D43.2 (A)
- new net: D10.2 (A), D9.1 (K)
- new net: R6.1, U3.10 (OUT)
- new net: R4.2, U3.2 (ISET)
- new net: R5.2, U3.4 (PRE-TERM)
- new net: C5.1, U1.4 (VCC)
- new net: R7.1, U1.5 (COMP)
- new net: D6.1 (K), D7.2 (A)
- new net: D227.1 (K), R34.1
- new net: D100.2 (A), D99.1 (K)
- new net: D226.1 (K), D227.2 (A)
- new net: D66.1 (K), D67.2 (A)
- new net BAT: C3.2, D1.2 (A), J1.1 (Pin_1), R6.2, SW1.3 (A)
- new net BAT_TEMP: J1.2 (Pin_2), U3.9 (TS)
- new net USB_D+: J2.A6 (D+), J2.B6 (D+), U3.5 (D+)
- new net USB_D-: J2.A7 (D-), J2.B7 (D-), U3.6 (D-)
- no-connect marks 0 -> 10
Other:
- note added: "Battery"
- note added: "Battery Charging"
- note added: "LED Driver"
- note added: "USB-C Receptacle"
- note removed: "Brightness Regulation"
- moved on the sheet: SW1

Commit message: Updated PCB
Parts:
- R1, R2, R3, R4, R5, R6: footprint (none) -> Resistor_SMD:R_0201_0603Metric
- SW1: footprint Button_Switch_THT:SW_NKK_G1xJP -> Button_Switch_THT:SW_Slide-03_Wuerth-WS-SLTV_10x2.5x6.4_P2.54mm
- U1: footprint (none) -> Package_SON:WSON-8-1EP_2x2mm_P0.5mm_EP0.9x1.6mm_ThermalVias
- U3: footprint (none) -> Package_SON:WSON-10-1EP_2.5x2.5mm_P0.5mm_EP1.2x2mm_ThermalVias
Changed lines of the file:
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@@
 			)
 		)
-		(property "Footprint" ""
+		(property "Footprint" "Resistor_SMD:R_0201_0603Metric"
 			(at 54.61 37.338 90)
 			(effects
@@
 			)
 		)
-		(property "Footprint" ""
+		(property "Footprint" "Package_SON:WSON-10-1EP_2.5x2.5mm_P0.5mm_EP1.2x2mm_ThermalVias"
 			(at 129.54 22.86 0)
 			(effects
@@
 			)
 		)
-		(property "Footprint" ""
+		(property "Footprint" "Package_SON:WSON-8-1EP_2x2mm_P0.5mm_EP0.9x1.6mm_ThermalVias"
 			(at 95.25 78.74 0)
 			(effects
@@
 			)
 		)
-		(property "Footprint" ""
+		(property "Footprint" "Resistor_SMD:R_0201_0603Metric"
 			(at 54.61 30.988 90)
 			(effects
@@
 			)
 		)
-		(property "Footprint" ""
+		(property "Footprint" "Resistor_SMD:R_0201_0603Metric"
 			(at 149.86 29.718 90)
 			(effects
@@
 			)
 		)
-		(property "Footprint" ""
+		(property "Footprint" "Resistor_SMD:R_0201_0603Metric"
 			(at 109.22 41.148 90)
 			(effects
@@
 			)
 		)
-		(property "Footprint" ""
+		(property "Footprint" "Resistor_SMD:R_0201_0603Metric"
 			(at 22.352 97.79 90)
 			(effects
@@
 			)
 		)
-		(property "Footprint" ""
+		(property "Footprint" "Resistor_SMD:R_0201_0603Metric"
 			(at 109.22 33.528 90)
 			(effects
@@
 			)
 		)
-		(property "Footprint" "Button_Switch_THT:SW_NKK_G1xJP"
+		(property "Footprint" "Button_Switch_THT:SW_Slide-03_Wuerth-WS-SLTV_10x2.5x6.4_P2.54mm"
 			(at 77.47 38.1 0)
 			(effects

Commit message: Final touches to PCB
Parts:
- RV1: footprint Potentiometer_THT:Potentiometer_Bourns_3296X_Horizontal -> Potentiometer_THT:Potentiometer_Bourns_3386P_Vertical
Changed lines of the file:
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@@
 			)
 		)
-		(property "Footprint" "Potentiometer_THT:Potentiometer_Bourns_3296X_Horizontal"
+		(property "Footprint" "Potentiometer_THT:Potentiometer_Bourns_3386P_Vertical"
 			(at 73.66 92.71 0)
 			(effects
